File: projects/blue-dream-space/build/blue-dream-space.kicad_pcb (KiCad board)
At the start: 4 copper layers, 347.5 x 172 mm, 181 parts, among them J1 USB_C, SW1 SW_Push, SW10 SW_Push, SW11 SW_Push, SW12 SW_Push, SW13 SW_Push, SW14 SW_Push, SW15 SW_Push, SW16 SW_Push, SW17 SW_Push, SW18 SW_Push, SW19 SW_Push, SW2 SW_Push, SW20 SW_Push, SW21 SW_Push, SW22 SW_Push, SW23 SW_Push, SW24 SW_Push, SW25 SW_Push, SW26 SW_Push, SW27 SW_Push, SW28 SW_Push, SW29 SW_Push, SW3 SW_Push, SW30 SW_Push, SW31 SW_Push, SW32 SW_Push, SW33 SW_Push, SW34 SW_Push, SW35 SW_Push, SW36 SW_Push, SW37 SW_Push, SW38 SW_Push, SW39 SW_Push, SW4 SW_Push, SW40 SW_Push, SW41 SW_Push, SW42 SW_Push, SW43 SW_Push, SW44 SW_Push, SW45 SW_Push, SW46 SW_Push, SW47 SW_Push, SW48 SW_Push, SW49 SW_Push, SW5 SW_Push, SW50 SW_Push, SW51 SW_Push, SW52 SW_Push, SW53 SW_Push, SW54 SW_Push, SW55 SW_Push, SW56 SW_Push, SW57 SW_Push, SW58 SW_Push, SW59 SW_Push, SW6 SW_Push, SW60 SW_Push, SW61 SW_Push, SW62 SW_Push, SW63 SW_Push, SW64 SW_Push, SW65 SW_Push, SW66 SW_Push, SW67 SW_Push, SW68 SW_Push, SW69 SW_Push, SW7 SW_Push, SW70 SW_Push, SW71 SW_Push, SW72 SW_Push, SW73 SW_Push, SW74 SW_Push, SW75 SW_Push, SW76 SW_Push, SW77 SW_Push, SW78 SW_Push, SW79 SW_Push, SW8 SW_Push, SW80 SW_Push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

Commit message: feat: major improvements across toolchain, web wizard, and routing
Build & Routing:
- Fix board outline to match layout editor (tight margin, no extra space)
- Add boardOutline override support for future polygon outlines
- Add copper zone fills (GND/VCC) on inner layers for 4-layer boards
- Fix USB connector rotation (180° for rear, port faces outward)
- Add power button footprint with auto-rotation toward nearest edge
- Fix layout override PCB_ORIGIN offset for all components
- Fix plate/case generators to respect screw position overrides
- Configurable max_passes and routing timeout in Build UI
- Freerouting: let it finish naturally (no kill), disable post-route optimization
- Freerouting: clean log output, strip job IDs and noisy warnings
- Freerouting: stream progress to web UI via SSE in real-time
- Fix freerouting.json CWD so gui.enabled=false is read
- Default timeout 10min, max passes 25

Web Wizard:
- Persist build state (stages, log, files) across tab navigation
- Add live elapsed timer per build stage, formatted duration on completion
- Add configurable routing passes and timeout inputs in Build tab
- Add fullscreen toggle for build log viewer
- Add output checkboxes in Build tab (independent from Config)
- Add last build timestamp display
- Fix config selection highlighting (flexible ID matching)
- Fix gerbers default to true
- Add charge current guidance with charger-specific limits
- Fix overview layout-editor status (shows customized count)
- Side-aware collision detection in layout editor (front/back/through)
- MCU and battery default to back side (under switches)
- Visual side badges (F/B/T) on layout editor components
- Undo/redo system for layout editor (Ctrl+Z/Ctrl+Shift+Z)
- Fix drag scaling for HiDPI displays
- Layout split ratio persisted to localStorage
- Remove app-content padding for full-width views

Data & Components:
- Add RP2040 Pro Micro, STM32F401 Black Pill, ESP32-S3 Mini MCUs
- Enrich all 25+ component files with features, concerns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
Parts:
- removed MH_bl, MH_br, MH_ml, MH_mr, MH_tr: MountingHole_M2.5, MountingHole:MountingHole_2.7mm_M2.5_Pad_Via
- added MH_screw_bl: MountingHole_M2.5, MountingHole:MountingHole_2.7mm_M2.5_Pad_Via, F.Cu at (22.5, 146.5)
- added MH_screw_br: MountingHole_M2.5, MountingHole:MountingHole_2.7mm_M2.5_Pad_Via, F.Cu at (357.0, 146.5)
- added MH_screw_ml: MountingHole_M2.5, MountingHole:MountingHole_2.7mm_M2.5_Pad_Via, F.Cu at (127.5, 45.5)
- added MH_screw_mr: MountingHole_M2.5, MountingHole:MountingHole_2.7mm_M2.5_Pad_Via, F.Cu at (281.5, 96.0)
- added MH_screw_tl: MountingHole_M2.5, MountingHole:MountingHole_2.7mm_M2.5_Pad_Via, F.Cu at (22.5, 22.5)
- added MH_screw_tr: MountingHole_M2.5, MountingHole:MountingHole_2.7mm_M2.5_Pad_Via, F.Cu at (357.0, 23.0)
- SW_PWR: renamed from MH_tl; value MountingHole_M2.5 -> Power; footprint MountingHole:MountingHole_2.7mm_M2.5_Pad_Via -> Button_Switch_SMD:SW_SPDT_CK-JS102011SAQN
- moved SW_PWR 204.7 mm to (330.5, 23.0), turned to 180 degrees
- moved BT1 122.4 mm to (331.0, 38.0), turned to 180 degrees
- moved J1 50.1 mm to (302.0, 23.0), turned to 180 degrees
- moved U1 24.3 mm to (181.5, 136.5)
Connections:
- SW_PWR pad 1: (no net) -> VBAT
Routing:
- net COL4: track 0.00 -> 519.1 mm, vias 0 -> 14
- net COL0: track 0.00 -> 517.7 mm, vias 0 -> 12
- net COL1: track 0.00 -> 517.4 mm, vias 0 -> 13
- net ROW10: track 0.00 -> 503.7 mm, vias 0 -> 10
- net COL7: track 0.00 -> 487.6 mm, vias 0 -> 11
- net COL6: track 0.00 -> 485.4 mm, vias 0 -> 14
- net COL5: track 0.00 -> 479.3 mm, vias 0 -> 14
- net COL2: track 0.00 -> 478.0 mm, vias 0 -> 14
- net COL3: track 0.00 -> 477.6 mm, vias 0 -> 14
- net ROW1: track 0.00 -> 395.6 mm, vias 0 -> 5
- net ROW0: track 0.00 -> 386.4 mm, vias 0 -> 5
- net ROW3: track 0.00 -> 382.7 mm, vias 0 -> 5
- net ROW5: track 0.00 -> 380.1 mm, vias 0 -> 5
- net ROW2: track 0.00 -> 378.2 mm, vias 0 -> 4
- net ROW4: track 0.00 -> 360.9 mm, vias 0 -> 3
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- added copper zone on B.Cu, net GND
- added copper zone on In1.Cu, net GND
- added copper zone on In2.Cu, net VCC
Other:
- board size 347.5 x 172 mm -> 347.5 x 137 mm
- net class Default removed
- net class Power removed

Commit message: feat: expanded component database, filterable selection UI, and PCB fixes
Component Database Expansion:
- MCUs: 8 → 21 (Liatris, Pillbug, Puchi-BLE, Splinky, STM32F072, STM32F411,
  STM32WB55, nRF52833, CH552, CH582, KB2040, WeAct RP2040, XIAO RP2040)
- Switches: 5 → 11 (Kailh BOX, Kailh Speed, Outemu LP, Akko CS, Gateron MX, Outemu MX)
- All components enriched with full specs: flash, RAM, clock, voltage, dimensions,
  split support, firmware support, activation/travel distance, total height, profile

Config UI — Filterable Component Selection:
- New ComponentFilter.tsx with dynamic dropdowns populated from component data
- New ComponentListItem.tsx with expandable spec tables, variant lists, supplier links
- Filter types: select, boolean, range brackets, multi-select, max price (numeric input)
- Switch filters: type, brand, profile, hotswap, mounting, actuation, travel, height, price
- MCU filters: USB, BLE, BLE version, charger, split, firmware, GPIOs, voltage, flash, RAM, clock, price
- Empty filter options removed, case-insensitive multi-match
- Click row to select, "See Details" toggle, styled "View →" button

PCB Generator Fixes:
- Fix KiCad 9 "Failed to load board" — vias no longer include "*.Mask" layer
- Separate viaCopperLayers (copper only) from allCopperLayers (copper + mask)
- Per-key RGB LEDs now on F.Cu (top side with switches), not B.Cu
- Clearance increased to 0.25mm for cleaner QFN routing
- MCU fanout vias option for 4-layer boards with collision-aware layout editor outline
- RGB underglow: 12 LEDs placed around PCB perimeter on B.Cu
- Routing guide updated: LEDs on correct layers, copper fill descriptions

Features Config:
- Detailed descriptions for all feature options (per-key RGB, underglow, encoder, OLED)
- LED placement labels fixed: "Below switch (south)" / "Above switch (north)"
- LED placement radio buttons shown inline

Co-Authored-By: Claude Opus 4.6 (1M context) <noreply@anthropic.com>
Parts:
- removed the D12 at (258.4, 42.5)
- removed the D15 at (321.2, 42.5)
- removed the D22 at (129.8, 66.3)
- removed the D26 at (206.0, 66.3)
- removed the D29 at (263.1, 66.3)
- removed the D36 at (106.0, 85.4)
- removed the D43 at (239.3, 85.4)
- removed the D5 at (115.5, 42.5)
- removed the D51 at (91.7, 104.4)
- removed the D8 at (177.4, 42.5)
- removed the SW11 at (239.3, 34.5)
- removed the SW18 at (53.6, 58.3)
- removed the SW25 at (186.9, 58.3)
- removed the SW29 at (263.1, 58.3)
- removed the SW32 at (345.2, 58.3)
- removed the SW36 at (106.0, 77.4)
- removed the SW39 at (163.1, 77.4)
- removed the SW4 at (96.4, 34.5)
- removed the SW43 at (239.3, 77.4)
- removed the SW46 at (301.2, 86.9)
- removed the SW52 at (110.7, 96.4)
- removed the SW8 at (177.4, 34.5)
- added BT1: Battery, Connector_JST:JST_PH_S2B-PH-K_1x02_P2.00mm_Horizontal, F.Cu at (331.0, 38.0)
- added D14: 1N4148, Diode_SMD:D_SOD-123, F.Cu at (302.2, 42.5)
- added D20: 1N4148, Diode_SMD:D_SOD-123, F.Cu at (91.7, 66.3)
- added D27: 1N4148, Diode_SMD:D_SOD-123, F.Cu at (225.0, 66.3)
- added D32: 1N4148, Diode_SMD:D_SOD-123, F.Cu at (345.2, 66.3)
- added D45: 1N4148, Diode_SMD:D_SOD-123, F.Cu at (277.4, 85.4)
- added D46: 1N4148, Diode_SMD:D_SOD-123, F.Cu at (301.2, 94.9)
- added D58: 1N4148, Diode_SMD:D_SOD-123, F.Cu at (225.0, 104.4)
- added D59: 1N4148, Diode_SMD:D_SOD-123, F.Cu at (244.1, 104.4)
- added D6: 1N4148, Diode_SMD:D_SOD-123, F.Cu at (139.3, 42.5)
- added D66: 1N4148, Diode_SMD:D_SOD-123, F.Cu at (115.5, 123.5)
- added D7: 1N4148, Diode_SMD:D_SOD-123, F.Cu at (158.3, 42.5)
- added D71: 1N4148, Diode_SMD:D_SOD-123, F.Cu at (210.7, 123.5)
- added D72: 1N4148, Diode_SMD:D_SOD-123, F.Cu at (229.8, 123.5)
- added D79: 1N4148, Diode_SMD:D_SOD-123, F.Cu at (84.5, 142.5)
- added D84: 1N4148, Diode_SMD:D_SOD-123, F.Cu at (306.0, 142.5)
- added D85: 1N4148, Diode_SMD:D_SOD-123, F.Cu at (325.0, 142.5)
- added J1: USB_C, Connector_USB:USB_C_Receptacle_GCT_USB4085, F.Cu at (302.0, 23.0)
- added LED10: SK6812MINI-E, LED_SMD:LED_SK6812MINI-E, F.Cu at (220.3, 40.5)
- added LED12: SK6812MINI-E, LED_SMD:LED_SK6812MINI-E, F.Cu at (258.4, 40.5)
- added LED13: SK6812MINI-E, LED_SMD:LED_SK6812MINI-E, F.Cu at (277.4, 40.5)
- added LED14: SK6812MINI-E, LED_SMD:LED_SK6812MINI-E, F.Cu at (302.2, 40.5)
- added LED16: SK6812MINI-E, LED_SMD:LED_SK6812MINI-E, F.Cu at (340.3, 40.5)
- added LED17: SK6812MINI-E, LED_SMD:LED_SK6812MINI-E, F.Cu at (34.5, 64.3)
- added LED19: SK6812MINI-E, LED_SMD:LED_SK6812MINI-E, F.Cu at (72.6, 64.3)
- added LED2: SK6812MINI-E, LED_SMD:LED_SK6812MINI-E, F.Cu at (58.3, 40.5)
- added LED20: SK6812MINI-E, LED_SMD:LED_SK6812MINI-E, F.Cu at (91.7, 64.3)
- added LED21: SK6812MINI-E, LED_SMD:LED_SK6812MINI-E, F.Cu at (110.7, 64.3)
- added LED23: SK6812MINI-E, LED_SMD:LED_SK6812MINI-E, F.Cu at (148.8, 64.3)
- added LED24: SK6812MINI-E, LED_SMD:LED_SK6812MINI-E, F.Cu at (167.9, 64.3)
- added LED26: SK6812MINI-E, LED_SMD:LED_SK6812MINI-E, F.Cu at (206.0, 64.3)
- added LED27: SK6812MINI-E, LED_SMD:LED_SK6812MINI-E, F.Cu at (225.0, 64.3)
- added LED28: SK6812MINI-E, LED_SMD:LED_SK6812MINI-E, F.Cu at (244.1, 64.3)
- added LED3: SK6812MINI-E, LED_SMD:LED_SK6812MINI-E, F.Cu at (77.4, 40.5)
- added LED30: SK6812MINI-E, LED_SMD:LED_SK6812MINI-E, F.Cu at (294.1, 64.3)
- added LED31: SK6812MINI-E, LED_SMD:LED_SK6812MINI-E, F.Cu at (326.2, 64.3)
- added LED33: SK6812MINI-E, LED_SMD:LED_SK6812MINI-E, F.Cu at (41.7, 83.4)
- added LED34: SK6812MINI-E, LED_SMD:LED_SK6812MINI-E, F.Cu at (67.9, 83.4)
- added LED35: SK6812MINI-E, LED_SMD:LED_SK6812MINI-E, F.Cu at (86.9, 83.4)
- added LED37: SK6812MINI-E, LED_SMD:LED_SK6812MINI-E, F.Cu at (125.0, 83.4)
- added LED38: SK6812MINI-E, LED_SMD:LED_SK6812MINI-E, F.Cu at (144.1, 83.4)
- added LED40: SK6812MINI-E, LED_SMD:LED_SK6812MINI-E, F.Cu at (182.2, 83.4)
- added LED41: SK6812MINI-E, LED_SMD:LED_SK6812MINI-E, F.Cu at (201.2, 83.4)
- added LED42: SK6812MINI-E, LED_SMD:LED_SK6812MINI-E, F.Cu at (220.3, 83.4)
- added LED44: SK6812MINI-E, LED_SMD:LED_SK6812MINI-E, F.Cu at (258.4, 83.4)
- added LED45: SK6812MINI-E, LED_SMD:LED_SK6812MINI-E, F.Cu at (277.4, 83.4)
- added LED47: SK6812MINI-E, LED_SMD:LED_SK6812MINI-E, F.Cu at (326.2, 83.4)
- added LED48: SK6812MINI-E, LED_SMD:LED_SK6812MINI-E, F.Cu at (345.2, 83.4)
- added LED49: SK6812MINI-E, LED_SMD:LED_SK6812MINI-E, F.Cu at (44.0, 102.4)
- added LED5: SK6812MINI-E, LED_SMD:LED_SK6812MINI-E, F.Cu at (115.5, 40.5)
- added LED50: SK6812MINI-E, LED_SMD:LED_SK6812MINI-E, F.Cu at (72.6, 102.4)
- added LED51: SK6812MINI-E, LED_SMD:LED_SK6812MINI-E, F.Cu at (91.7, 102.4)
- added LED52: SK6812MINI-E, LED_SMD:LED_SK6812MINI-E, F.Cu at (110.7, 102.4)
- added LED54: SK6812MINI-E, LED_SMD:LED_SK6812MINI-E, F.Cu at (148.8, 102.4)
- added LED55: SK6812MINI-E, LED_SMD:LED_SK6812MINI-E, F.Cu at (167.9, 102.4)
- added LED56: SK6812MINI-E, LED_SMD:LED_SK6812MINI-E, F.Cu at (186.9, 102.4)
- added LED57: SK6812MINI-E, LED_SMD:LED_SK6812MINI-E, F.Cu at (206.0, 102.4)
- added LED58: SK6812MINI-E, LED_SMD:LED_SK6812MINI-E, F.Cu at (225.0, 102.4)
- added LED59: SK6812MINI-E, LED_SMD:LED_SK6812MINI-E, F.Cu at (244.1, 102.4)
- added LED6: SK6812MINI-E, LED_SMD:LED_SK6812MINI-E, F.Cu at (139.3, 40.5)
- added LED60: SK6812MINI-E, LED_SMD:LED_SK6812MINI-E, F.Cu at (263.1, 102.4)
- added LED61: SK6812MINI-E, LED_SMD:LED_SK6812MINI-E, F.Cu at (326.2, 102.4)
- added LED62: SK6812MINI-E, LED_SMD:LED_SK6812MINI-E, F.Cu at (345.2, 102.4)
- added LED63: SK6812MINI-E, LED_SMD:LED_SK6812MINI-E, F.Cu at (46.4, 121.5)
- added LED64: SK6812MINI-E, LED_SMD:LED_SK6812MINI-E, F.Cu at (77.4, 121.5)
- added LED65: SK6812MINI-E, LED_SMD:LED_SK6812MINI-E, F.Cu at (96.4, 121.5)
- added LED66: SK6812MINI-E, LED_SMD:LED_SK6812MINI-E, F.Cu at (115.5, 121.5)
- added LED67: SK6812MINI-E, LED_SMD:LED_SK6812MINI-E, F.Cu at (134.5, 121.5)
- added LED68: SK6812MINI-E, LED_SMD:LED_SK6812MINI-E, F.Cu at (153.6, 121.5)
- added LED69: SK6812MINI-E, LED_SMD:LED_SK6812MINI-E, F.Cu at (172.6, 121.5)
- added LED7: SK6812MINI-E, LED_SMD:LED_SK6812MINI-E, F.Cu at (158.3, 40.5)
- added LED70: SK6812MINI-E, LED_SMD:LED_SK6812MINI-E, F.Cu at (191.7, 121.5)
- added LED71: SK6812MINI-E, LED_SMD:LED_SK6812MINI-E, F.Cu at (210.7, 121.5)
- added LED72: SK6812MINI-E, LED_SMD:LED_SK6812MINI-E, F.Cu at (229.8, 121.5)
- added LED73: SK6812MINI-E, LED_SMD:LED_SK6812MINI-E, F.Cu at (248.8, 121.5)
- added LED74: SK6812MINI-E, LED_SMD:LED_SK6812MINI-E, F.Cu at (275.0, 121.5)
- added LED75: SK6812MINI-E, LED_SMD:LED_SK6812MINI-E, F.Cu at (306.0, 121.5)
- added LED76: SK6812MINI-E, LED_SMD:LED_SK6812MINI-E, F.Cu at (346.9, 123.4)
- added LED77: SK6812MINI-E, LED_SMD:LED_SK6812MINI-E, F.Cu at (36.9, 140.5)
- added LED78: SK6812MINI-E, LED_SMD:LED_SK6812MINI-E, F.Cu at (60.7, 140.5)
- added LED79: SK6812MINI-E, LED_SMD:LED_SK6812MINI-E, F.Cu at (84.5, 140.5)
- added LED80: SK6812MINI-E, LED_SMD:LED_SK6812MINI-E, F.Cu at (158.3, 140.5)
- added LED81: SK6812MINI-E, LED_SMD:LED_SK6812MINI-E, F.Cu at (232.2, 140.5)
- added LED82: SK6812MINI-E, LED_SMD:LED_SK6812MINI-E, F.Cu at (256.0, 140.5)
- added LED83: SK6812MINI-E, LED_SMD:LED_SK6812MINI-E, F.Cu at (286.9, 140.5)
- added LED84: SK6812MINI-E, LED_SMD:LED_SK6812MINI-E, F.Cu at (306.0, 140.5)
- added LED85: SK6812MINI-E, LED_SMD:LED_SK6812MINI-E, F.Cu at (325.0, 140.5)
- added LED86: SK6812MINI-E, LED_SMD:LED_SK6812MINI-E, F.Cu at (346.9, 142.4)
- added LED9: SK6812MINI-E, LED_SMD:LED_SK6812MINI-E, F.Cu at (196.4, 40.5)
- added MH_screw_br: MountingHole_M2.5, MountingHole:MountingHole_2.7mm_M2.5_Pad_Via, F.Cu at (357.0, 146.5)
- added MH_screw_ml: MountingHole_M2.5, MountingHole:MountingHole_2.7mm_M2.5_Pad_Via, F.Cu at (127.5, 45.5)
- added SW14: SW_Push, Switch:SW_Push, F.Cu at (302.2, 34.5)
- added SW2: SW_Push, Switch:SW_Push, F.Cu at (58.3, 34.5)
- added SW27: SW_Push, Switch:SW_Push, F.Cu at (225.0, 58.3)
- added SW28: SW_Push, Switch:SW_Push, F.Cu at (244.1, 58.3)
- added SW35: SW_Push, Switch:SW_Push, F.Cu at (86.9, 77.4)
- added SW40: SW_Push, Switch:SW_Push, F.Cu at (182.2, 77.4)
- added SW41: SW_Push, Switch:SW_Push, F.Cu at (201.2, 77.4)
- added SW48: SW_Push, Switch:SW_Push, F.Cu at (345.2, 77.4)
- added SW53: SW_Push, Switch:SW_Push, F.Cu at (129.8, 96.4)
- added SW54: SW_Push, Switch:SW_Push, F.Cu at (148.8, 96.4)
- added SW61: SW_Push, Switch:SW_Push, F.Cu at (326.2, 96.4)
- added SW66: SW_Push, Switch:SW_Push, F.Cu at (115.5, 115.5)
- added SW67: SW_Push, Switch:SW_Push, F.Cu at (134.5, 115.5)
- added SW74: SW_Push, Switch:SW_Push, F.Cu at (275.0, 115.5)
- added SW79: SW_Push, Switch:SW_Push, F.Cu at (84.5, 134.5)
- added SW80: SW_Push, Switch:SW_Push, F.Cu at (158.3, 134.5)
- added SW9: SW_Push, Switch:SW_Push, F.Cu at (196.4, 34.5)
- D12: renamed from SW22; value SW_Push -> 1N4148; footprint Switch:SW_Push -> Diode_SMD:D_SOD-123
- D19: renamed from SW35; value SW_Push -> 1N4148; footprint Switch:SW_Push -> Diode_SMD:D_SOD-123
- D26: renamed from SW48; value SW_Push -> 1N4148; footprint Switch:SW_Push -> Diode_SMD:D_SOD-123
- D33: renamed from SW61; value SW_Push -> 1N4148; footprint Switch:SW_Push -> Diode_SMD:D_SOD-123
- D40: renamed from SW74; value SW_Push -> 1N4148; footprint Switch:SW_Push -> Diode_SMD:D_SOD-123
- D5: renamed from SW9; value SW_Push -> 1N4148; footprint Switch:SW_Push -> Diode_SMD:D_SOD-123
- D51: renamed from J1; value USB_C -> 1N4148; footprint Connector_USB:USB_C_Receptacle_GCT_USB4085 -> Diode_SMD:D_SOD-123
- D53: renamed from MH_screw_br; value MountingHole_M2.5 -> 1N4148; footprint MountingHole:MountingHole_2.7mm_M2.5_Pad_Via -> Diode_SMD:D_SOD-123
- LED1: renamed from SW2; value SW_Push -> SK6812MINI-E; footprint Switch:SW_Push -> LED_SMD:LED_SK6812MINI-E
- LED11: renamed from D20; value 1N4148 -> SK6812MINI-E; footprint Diode_SMD:D_SOD-123 -> LED_SMD:LED_SK6812MINI-E
- LED15: renamed from SW28; value SW_Push -> SK6812MINI-E; footprint Switch:SW_Push -> LED_SMD:LED_SK6812MINI-E
- LED18: renamed from D33; value 1N4148 -> SK6812MINI-E; footprint Diode_SMD:D_SOD-123 -> LED_SMD:LED_SK6812MINI-E
- LED22: renamed from SW41; value SW_Push -> SK6812MINI-E; footprint Switch:SW_Push -> LED_SMD:LED_SK6812MINI-E
- LED25: renamed from D46; value 1N4148 -> SK6812MINI-E; footprint Diode_SMD:D_SOD-123 -> LED_SMD:LED_SK6812MINI-E
- LED29: renamed from SW54; value SW_Push -> SK6812MINI-E; footprint Switch:SW_Push -> LED_SMD:LED_SK6812MINI-E
- LED32: renamed from D59; value 1N4148 -> SK6812MINI-E; footprint Diode_SMD:D_SOD-123 -> LED_SMD:LED_SK6812MINI-E
- LED36: renamed from SW67; value SW_Push -> SK6812MINI-E; footprint Switch:SW_Push -> LED_SMD:LED_SK6812MINI-E
- LED39: renamed from D72; value 1N4148 -> SK6812MINI-E; footprint Diode_SMD:D_SOD-123 -> LED_SMD:LED_SK6812MINI-E
- LED4: renamed from D7; value 1N4148 -> SK6812MINI-E; footprint Diode_SMD:D_SOD-123 -> LED_SMD:LED_SK6812MINI-E
- LED43: renamed from SW80; value SW_Push -> SK6812MINI-E; footprint Switch:SW_Push -> LED_SMD:LED_SK6812MINI-E
- LED46: renamed from D85; value 1N4148 -> SK6812MINI-E; footprint Diode_SMD:D_SOD-123 -> LED_SMD:LED_SK6812MINI-E
- LED53: renamed from MH_screw_ml; value MountingHole_M2.5 -> SK6812MINI-E; footprint MountingHole:MountingHole_2.7mm_M2.5_Pad_Via -> LED_SMD:LED_SK6812MINI-E
- LED8: renamed from SW15; value SW_Push -> SK6812MINI-E; footprint Switch:SW_Push -> LED_SMD:LED_SK6812MINI-E
- SW11: renamed from D19; value 1N4148 -> SW_Push; footprint Diode_SMD:D_SOD-123 -> Switch:SW_Push
- SW18: renamed from D32; value 1N4148 -> SW_Push; footprint Diode_SMD:D_SOD-123 -> Switch:SW_Push
- SW25: renamed from D45; value 1N4148 -> SW_Push; footprint Diode_SMD:D_SOD-123 -> Switch:SW_Push
- SW32: renamed from D58; value 1N4148 -> SW_Push; footprint Diode_SMD:D_SOD-123 -> Switch:SW_Push
- SW39: renamed from D71; value 1N4148 -> SW_Push; footprint Diode_SMD:D_SOD-123 -> Switch:SW_Push
- SW4: renamed from D6; value 1N4148 -> SW_Push; footprint Diode_SMD:D_SOD-123 -> Switch:SW_Push
- SW46: renamed from D84; value 1N4148 -> SW_Push; footprint Diode_SMD:D_SOD-123 -> Switch:SW_Push
- SW52: renamed from BT1; value Battery -> SW_Push; footprint Connector_JST:JST_PH_S2B-PH-K_1x02_P2.00mm_Horizontal -> Switch:SW_Push
- moved SW18 291.8 mm to (53.6, 58.3)
- moved D33 284.7 mm to (41.7, 85.4)
- moved D53 231.1 mm to (129.8, 104.4)
- moved SW52 227.9 mm to (110.7, 96.4), turned to 0 degrees
- moved D51 225.5 mm to (91.7, 104.4), turned to 0 degrees
- moved SW11 169.7 mm to (239.3, 34.5)
- moved D43 165.0 mm to (239.3, 85.4)
- moved SW43 165.0 mm to (239.3, 77.4)
- moved LED11 149.9 mm to (239.3, 40.5)
- moved LED8 144.0 mm to (177.4, 40.5)
- moved D26 139.7 mm to (206.0, 66.3)
- moved D29 138.7 mm to (263.1, 66.3)
- moved SW29 138.7 mm to (263.1, 58.3)
- moved D12 129.6 mm to (258.4, 42.5)
- moved SW32 128.7 mm to (345.2, 58.3)
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- renumbered D27 to D15, D40 to D22, D53 to D29, D66 to D36, D79 to D43, D14 to D8, SW27 to SW15, SW40 to SW22, SW53 to SW29, SW66 to SW36, SW79 to SW43, SW14 to SW8
Connections:
- D12 pad 1: COL5 -> ROW1
- D12 pad 2: ROW2 -> COL3
- D15 pad 1: ROW3 -> ROW1
- D15 pad 2: COL2 -> COL6
- D19 pad 1: COL2 -> ROW2
- D19 pad 2: ROW4 -> COL2
- D22 pad 1: ROW4 -> ROW2
- D22 pad 2: COL7 -> COL5
- D26 pad 1: COL7 -> ROW3
- D26 pad 2: ROW5 -> COL1
- D29 pad 1: ROW6 -> ROW3
- D33 pad 1: COL5 -> ROW4
- D33 pad 2: ROW7 -> COL0
- D36 pad 1: ROW8 -> ROW4
- D40 pad 1: COL4 -> ROW4
- D40 pad 2: ROW9 -> COL7
- D43 pad 1: ROW10 -> ROW5
- D5 pad 1: COL0 -> ROW0
- D5 pad 2: ROW1 -> COL4
- D53 pad 1: (no net) -> ROW6
- D8 pad 1: ROW1 -> ROW0
- D8 pad 2: COL5 -> COL7
- LED1 pad 1: COL1 -> VCC
- LED1 pad 2: ROW0 -> (no net)
- LED11 pad 1: ROW2 -> VCC
- LED11 pad 2: COL3 -> (no net)
- LED15 pad 1: COL3 -> VCC
- LED15 pad 2: ROW3 -> (no net)
- LED18 pad 1: ROW4 -> VCC
- LED18 pad 2: COL0 -> (no net)
- LED22 pad 1: COL0 -> VCC
- LED22 pad 2: ROW5 -> (no net)
- LED25 pad 1: ROW5 -> VCC
- LED25 pad 2: COL5 -> (no net)
- LED29 pad 1: COL5 -> VCC
- LED29 pad 2: ROW6 -> (no net)
- LED32 pad 1: ROW7 -> VCC
- LED32 pad 2: COL3 -> (no net)
- LED36 pad 1: COL4 -> VCC
- LED36 pad 2: ROW8 -> (no net)
- LED39 pad 1: ROW9 -> VCC
- LED39 pad 2: COL2 -> (no net)
- LED4 pad 1: ROW0 -> VCC
- LED4 pad 2: COL6 -> (no net)
- LED43 pad 1: COL3 -> VCC
- LED43 pad 2: ROW10 -> (no net)
- LED46 pad 1: ROW10 -> VCC
- LED46 pad 2: COL8 -> (no net)
- LED53 pad 1: (no net) -> VCC
- LED8 pad 1: COL6 -> VCC
- LED8 pad 2: ROW1 -> (no net)
- SW11 pad 1: ROW2 -> COL2
- SW11 pad 2: COL2 -> ROW1
- SW15 pad 1: COL2 -> COL6
- SW15 pad 2: ROW3 -> ROW1
- SW18 pad 1: ROW3 -> COL1
- SW18 pad 2: COL7 -> ROW2
- SW22 pad 1: COL7 -> COL5
- SW22 pad 2: ROW4 -> ROW2
- SW25 pad 1: ROW5 -> COL0
- SW25 pad 2: COL4 -> ROW3
- SW29 pad 2: ROW6 -> ROW3
- SW32 pad 1: ROW7 -> COL7
- SW32 pad 2: COL2 -> ROW3
- SW36 pad 2: ROW8 -> ROW4
- SW39 pad 1: ROW9 -> COL6
- SW39 pad 2: COL1 -> ROW4
- SW4 pad 1: ROW0 -> COL3
- SW4 pad 2: COL5 -> ROW0
- SW43 pad 2: ROW10 -> ROW5
- SW46 pad 1: ROW10 -> COL5
- SW46 pad 2: COL7 -> ROW5
- SW52 pad 1: VBAT -> COL3
- SW52 pad 2: GND -> ROW6
- SW8 pad 1: COL5 -> COL7
- SW8 pad 2: ROW1 -> ROW0
Routing:
- net COL4: track 519.1 -> 1.20 mm, vias 14 -> 1
- net COL0: track 517.7 -> 1.20 mm, vias 12 -> 1
- net COL1: track 517.4 -> 1.20 mm, vias 13 -> 1
- net ROW10: track 503.7 -> 1.20 mm, vias 10 -> 1
- net COL7: track 487.6 -> 1.20 mm, vias 11 -> 1
- net COL6: track 485.4 -> 1.20 mm, vias 14 -> 1
- net COL5: track 479.3 -> 1.20 mm, vias 14 -> 1
- net COL2: track 478.0 -> 1.20 mm, vias 14 -> 1
- net COL3: track 477.6 -> 1.20 mm, vias 14 -> 1
- net ROW1: track 395.6 -> 1.20 mm, vias 5 -> 1
- net ROW0: track 386.4 -> 1.20 mm, vias 5 -> 1
- net ROW3: track 382.7 -> 1.20 mm, vias 5 -> 1
- net ROW5: track 380.1 -> 1.20 mm, vias 5 -> 1
- net ROW2: track 378.2 -> 1.20 mm, vias 4 -> 1
- net ROW4: track 360.9 -> 1.20 mm, vias 3 -> 1
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Other:
- net class Default added: clearance 0.25, trace_width 0.2, via_dia 0.6, via_drill 0.3
- net class Power added: clearance 0.25, trace_width 0.4, via_dia 0.8, via_drill 0.4
- rule pad_to_mask_clearance: 0.025 -> 0.05
- rule solder_mask_min_width: 0.05 -> 0.1

Commit message: feat: data-driven MCU footprints, fanout fix, routing helpers, gerber fix
- Fix KiCad 9 gerber export: vias use start/end layers only (not all 4)
- Fix layout path resolution in orchestrator (relative to project dir)
- Refactor MCU footprint generation to be data-driven from component DB
  - New mcu-footprint.ts: bare-chip (QFN/QFP) and module (DIP) generators
  - Staggered fanout vias (inner/outer rows) to prevent overlap at 0.5mm pitch
  - Fanout now includes VCC, GND, USB nets (not just GPIOs)
  - Modules get through-hole footprint, bare chips get SMD with optional fanout
  - Graceful fallback with warnings for unknown MCUs
- Add verified boardPins data for all 21 MCUs from official datasheets/firmware
  - Pro-micro: nice!nano, KB2040, Liatris, Splinky, Puchi-BLE, SparkFun, SuperMini
  - BlackPill: STM32F401, STM32F411, PillBug (reclassified from pro-micro)
  - XIAO: XIAO BLE, XIAO RP2040
  - Pico: WeAct RP2040
  - Castellated: Holyiot 18010, ESP32-S3 Mini
  - Bare chips: CH552T, CH582M, nRF52833, STM32F072, STM32WB55 (package+pinMap)
- Fix nice!nano boardPins: 21 GPIOs (was 16, missing D8/D9/bottom pads)
- Fix STM32WB55 gpioCount: 42 (was incorrectly 48)
- Add routing helper message after build for manual/incomplete routing
  - Shows Freerouting command with correct paths from repo root
  - Explains -mp (max passes) and -mt (optimization threads)
  - Documents freerouting.json config location
  - Shows gerber re-export commands
- DSN now always exported (even manual/guided mode) for later Freerouting use
- routePCB returns RoutingResult with incomplete flag
- runFreerouting returns boolean (all routed vs unrouted remaining)
- Freerouting jar finder prefers highest version (v2.1.0 over v1.9.0)
- Hide complex nested objects (boardPins, pinMap) from component detail UI
- Add McuData, McuPackage, McuPinMap, McuBoardPins types

Co-Authored-By: Claude Opus 4.6 (1M context) <noreply@anthropic.com>
Parts:
- U1: value nRF52840 -> nice!nano v2; footprint Package_DFN_QFN:QFN-48-1EP_7x7mm_P0.5mm_EP5.6x5.6mm -> Module:pro-micro_29pin_P2.54mm
Connections:
- U1 pad 1: ROW0 -> VBAT
- U1 pad 10: ROW9 -> ROW5
- U1 pad 11: ROW10 -> ROW6
- U1 pad 12: COL0 -> ROW7
- U1 pad 13: COL1 -> VBUS
- U1 pad 14: COL2 -> GND
- U1 pad 15: COL3 -> (no net)
- U1 pad 16: COL4 -> VCC
- U1 pad 17: COL5 -> ROW8
- U1 pad 18: COL6 -> ROW9
- U1 pad 19: COL7 -> ROW10
- U1 pad 2: ROW1 -> GND
- U1 pad 20: COL8 -> COL0
- U1 pad 21: COL9 -> COL1
- U1 pad 22: (no net) -> COL2
- U1 pad 23: (no net) -> COL3
- U1 pad 24: (no net) -> COL4
- U1 pad 25: (no net) -> COL5
- U1 pad 26: (no net) -> COL6
- U1 pad 27: (no net) -> COL7
- U1 pad 28: (no net) -> COL8
- U1 pad 29: (no net) -> COL9
- U1 pad 3: ROW2 -> (no net)
- U1 pad 4: ROW3 -> VCC
- U1 pad 5: ROW4 -> ROW0
- U1 pad 6: ROW5 -> ROW1
- U1 pad 7: ROW6 -> ROW2
- U1 pad 8: ROW7 -> ROW3
- U1 pad 9: ROW8 -> ROW4
Routing:
- net ROW9: track 1.20 -> 0.00 mm, vias 1 -> 0
- net ROW8: track 1.20 -> 0.00 mm, vias 1 -> 0
- net ROW7: track 1.20 -> 0.00 mm, vias 1 -> 0
- net ROW6: track 1.20 -> 0.00 mm, vias 1 -> 0
- net ROW5: track 1.20 -> 0.00 mm, vias 1 -> 0
- net ROW4: track 1.20 -> 0.00 mm, vias 1 -> 0
- net ROW3: track 1.20 -> 0.00 mm, vias 1 -> 0
- net ROW2: track 1.20 -> 0.00 mm, vias 1 -> 0
- net ROW10: track 1.20 -> 0.00 mm, vias 1 -> 0
- net ROW1: track 1.20 -> 0.00 mm, vias 1 -> 0
- net ROW0: track 1.20 -> 0.00 mm, vias 1 -> 0
- net COL9: track 1.20 -> 0.00 mm, vias 1 -> 0
- net COL8: track 1.20 -> 0.00 mm, vias 1 -> 0
- net COL7: track 1.20 -> 0.00 mm, vias 1 -> 0
- net COL6: track 1.20 -> 0.00 mm, vias 1 -> 0
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
Commit message: feat: auto-routing env flag, zip download, MCU/charger fanout, layout editor polish
Server features:
- Add ENABLE_AUTO_ROUTING env flag to disable Freerouting on public deployments
- New /api/config/server endpoint exposes server capabilities to client
- New /api/build/:name/download endpoint zips entire build folder for download
- Cache zip archive in build folder, auto-invalidate when build files change
- Execution engine auto-switches to manual routing if auto-routing disabled
- File scanner excludes build-archive.zip from listing

Client features:
- "Download All Files" button in Build Output header
- Config page hides auto-route option when server doesn't support it
- Dynamic routing mode dropdown based on server config
- Hide complex nested objects (boardPins, pinMap) from component detail UI

Layout Editor:
- Data-driven component sizing from actual MCU/battery/charger/connector data
- Proper MCU dimensions from boardPins (modules) or package info (bare chips)
- Out-of-bounds detection with red outline for draggable components
- Right-side Properties panel with board side selector (front/back/through)
- Charger IC component in layout editor with data-driven sizing
- Charger fanout zone visualization for QFN chargers
- Battery color changed from red (looked invalid) to amber
- Arrow key Ctrl modifier for 0.1mm fine nudging (shift=0.25mm, default=1mm)
- Tip bar updated with all nudge modes

PCB generator:
- Charger IC footprint generation with packageInfo from data files
- Staggered charger fanout vias for QFN chargers on 4-layer boards
- Exposed thermal pad support for QFN chargers
- Uses footprintRef from charger data for accurate KiCad footprints

MCU data:
- Added verified boardPins for all 20 modules (from ZMK/QMK sources)
- Added pinMap and package info for all 6 bare chip MCUs
- Fixed nice!nano boardPins to include all 21 GPIOs (D8/D9/bottom pads)
- Fixed STM32WB55 gpioCount mismatch
- PillBug reclassified from pro-micro to blackpill form factor

Charger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
Parts:
- added SW_PWR: Power, Button_Switch_SMD:SW_SPDT_CK-JS102011SAQN, F.Cu at (330.5, 23.0)
- U2: renamed from SW_PWR; value Power -> bq24075; footprint Button_Switch_SMD:SW_SPDT_CK-JS102011SAQN -> Package_DFN_QFN:QFN-16-1EP_3.5x3.5mm_P0.5mm_EP2.15x2.15mm
- moved U2 144.6 mm to (204.9, 94.6), turned to 0 degrees
- moved BT1 38.3 mm to (335.5, 76.0)
- moved U1 10.0 mm to (183.5, 126.5)
Connections:
- U2 pad 1: VBAT -> VBUS
- U2 pad 2: VCC -> GND
- U2 pad 3: (no net) -> VBAT
Changed lines of the file:
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@@
   (footprint "Module:pro-micro_29pin_P2.54mm"
     (layer "F.Cu")
-    (at 182.5 136.5)
+    (at 183.5 126.5)
     (property "Reference" "U1" (at 0 -5) (layer "F.SilkS") (effects (font (size 1 1) (thickness 0.15))))
     (property "Value" "nice!nano v2" (at 0 5) (layer "F.Fab") (effects (font (size 1 1) (thickness 0.15))))
@@
   (footprint "Connector_JST:JST_PH_S2B-PH-K_1x02_P2.00mm_Horizontal"
     (layer "F.Cu")
-    (at 331 38 180)
+    (at 335.5 76 180)
     (property "Reference" "BT1" (at 0 -3) (layer "F.SilkS") (effects (font (size 1 1) (thickness 0.15))))
     (property "Value" "Battery" (at 0 3) (layer "F.Fab") (effects (font (size 1 1) (thickness 0.15))))
@@
     (pad "2" thru_hole circle (at 2 0) (size 1.75 1.75) (drill 1.0) (layers "F.Cu" "In1.Cu" "In2.Cu" "B.Cu" "*.Mask") (net 23 "GND"))
   )
+  (footprint "Package_DFN_QFN:QFN-16-1EP_3.5x3.5mm_P0.5mm_EP2.15x2.15mm"
+    (layer "F.Cu")
+    (at 204.8777 94.6265)
+    (property "Reference" "U2" (at 0 -3) (layer "F.SilkS") (effects (font (size 0.8 0.8) (thickness 0.12))))
+    (property "Value" "bq24075" (at 0 3) (layer "F.Fab") (effects (font (size 0.8 0.8) (thickness 0.12))))
+    (pad "1" smd rect (at -1.1 -0.65) (size 0.6 0.4) (layers "F.Cu" "F.Paste" "F.Mask") (net 24 "VBUS"))
+    (pad "2" smd rect (at -1.1 0) (size 0.6 0.4) (layers "F.Cu" "F.Paste" "F.Mask") (net 23 "GND"))
+    (pad "3" smd rect (at -1.1 0.65) (size 0.6 0.4) (layers "F.Cu" "F.Paste" "F.Mask") (net 25 "VBAT"))
+    (pad "4" smd rect (at 1.1 0) (size 0.6 0.4) (layers "F.Cu" "F.Paste" "F.Mask") (net 22 "VCC"))
+    (pad "EP" smd rect (at 0 0) (size 2.15 2.15) (layers "F.Cu" "F.Paste" "F.Mask") (net 23 "GND"))
+    (fp_rect (start -2.75 -2.75) (end 2.75 2.75) (stroke (width 0.05) (type default)) (fill none) (layer "F.CrtYd"))
+  )
   (footprint "Button_Switch_SMD:SW_SPDT_CK-JS102011SAQN"
