File: projects/blue-dream-space/build/blue-dream-space.kicad_sch (KiCad schematic)
At the start: 175 parts, among them J1 USB_C, SW1 R0C0, SW10 R1C1, SW11 R1C2, SW12 R1C3, SW13 R1C4, SW14 R1C5, SW15 R1C6, SW16 R1C7, SW17 R2C0, SW18 R2C1, SW19 R2C2, SW2 R0C1, SW20 R2C3, SW21 R2C4, SW22 R2C5, SW23 R2C6, SW24 R2C7, SW25 R3C0, SW26 R3C1, SW27 R3C2, SW28 R3C3, SW29 R3C4, SW3 R0C2, SW30 R3C5, SW31 R3C6, SW32 R3C7, SW33 R4C0, SW34 R4C1, SW35 R4C2, SW36 R4C3, SW37 R4C4, SW38 R4C5, SW39 R4C6, SW4 R0C3, SW40 R4C7, SW41 R5C0, SW42 R5C1, SW43 R5C2, SW44 R5C3, SW45 R5C4, SW46 R5C5, SW47 R5C6, SW48 R5C7, SW49 R6C0, SW5 R0C4, SW50 R6C1, SW51 R6C2, SW52 R6C3, SW53 R6C4, SW54 R6C5, SW55 R6C6, SW56 R7C0, SW57 R7C1, SW58 R7C2, SW59 R7C3, SW6 R0C5, SW60 R7C4, SW61 R7C5, SW62 R7C6, SW63 R8C0, SW64 R8C1, SW65 R8C2, SW66 R8C3, SW67 R8C4, SW68 R8C5, SW69 R8C6, SW7 R0C6, SW70 R9C0, SW71 R9C1, SW72 R9C2, SW73 R9C3, SW74 R9C4, SW75 R9C5, SW76 R9C6, SW77 R10C0, SW78 R10C1, SW79 R10C2, SW8 R0C7, SW80 R10C3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

Commit message: refactor: design tokens, shared primitives, and architecture decomposition
Design system & styling (Phase A):
- Extend global.css with spacing/font/transition/z-index/chrome tokens
- Add success-soft, warning-soft, error-soft, accent-soft, border-strong colors
- Replace ~62 hardcoded hex colors across views with design tokens
- Apply transition duration tokens to components.css and shell.css
- Add utility classes (u-stack, u-text-muted, panel-heading, field-label, empty-state)
- Global *:focus-visible accent outline for keyboard users
- Global accent-color for native checkboxes/radios
- Toast container offset uses calc(--status-bar-height + space)
- Document CSS naming convention at top of global.css
- New utils/format.ts with formatBytes/formatDuration/formatDateTime/formatRelativeTime
- FileLink and Build.tsx migrated to shared format helpers
- LayoutEditor uses panel-heading class instead of duplicated inline styles

Shared primitives (Phase B):
- New Input component (label, hint, error, sizes, prefix/suffix, onEnter)
- New Checkbox component (label, description slot, sizes, switch variant)
- New EmptyState component (icon, title, message, actions, variants)
- Modal accepts size prop (sm/md/lg/xl) + scroll-shadow + aria + hideClose
- NewProject migrated to Input with hint/error states
- Build.tsx routing settings + output checkboxes use Input + Checkbox
- Overview/Build empty states use EmptyState

Theme infrastructure (Phase B):
- Light theme tokens defined under [data-theme="light"]
- prefers-color-scheme: light auto-activates when no override
- index.html pins data-theme="dark" preserving current appearance

Server helpers (Phase B):
- New server/utils/safe-path.ts with centralized path-traversal protection
- build.routes.ts file serving migrated to safePath()

Type safety (Phase B):
- New src/wizard/src/types/mcu.types.ts mirroring tools package types
- LayoutState ComponentDataSet replaces any with McuData/ComponentOption
- getMcuDimensions strongly typed
- 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
Parts:
- SW10: value R1C1 -> R0C9
- SW11: value R1C2 -> R0C10
- SW12: value R1C3 -> R0C11
- SW13: value R1C4 -> R0C12
- SW14: value R1C5 -> R0C13
- SW15: value R1C6 -> R0C14
- SW16: value R1C7 -> R0C15
- SW17: value R2C0 -> R1C0
- SW18: value R2C1 -> R1C1
- SW19: value R2C2 -> R1C2
- SW20: value R2C3 -> R1C3
- SW21: value R2C4 -> R1C4
- SW22: value R2C5 -> R1C5
- SW23: value R2C6 -> R1C6
- SW24: value R2C7 -> R1C7
- SW25: value R3C0 -> R1C8
- SW26: value R3C1 -> R1C9
- SW27: value R3C2 -> R1C10
- SW28: value R3C3 -> R1C11
- SW29: value R3C4 -> R1C12
- SW30: value R3C5 -> R1C13
- SW31: value R3C6 -> R1C14
- SW32: value R3C7 -> R1C15
- SW33: value R4C0 -> R2C0
- SW34: value R4C1 -> R2C1
- SW35: value R4C2 -> R2C2
- SW36: value R4C3 -> R2C3
- SW37: value R4C4 -> R2C4
- SW38: value R4C5 -> R2C5
- SW39: value R4C6 -> R2C6
- SW40: value R4C7 -> R2C7
- SW41: value R5C0 -> R2C8
- SW42: value R5C1 -> R2C9
- SW43: value R5C2 -> R2C10
- SW44: value R5C3 -> R2C11
- SW45: value R5C4 -> R2C12
- SW46: value R5C5 -> R2C13
- SW47: value R5C6 -> R2C14
- SW48: value R5C7 -> R2C15
- SW49: value R6C0 -> R3C0
- SW50: value R6C1 -> R3C1
- SW51: value R6C2 -> R3C2
- SW52: value R6C3 -> R3C3
- SW53: value R6C4 -> R3C4
- SW54: value R6C5 -> R3C5
- SW55: value R6C6 -> R3C6
- SW56: value R7C0 -> R3C7
- SW57: value R7C1 -> R3C8
- SW58: value R7C2 -> R3C9
- SW59: value R7C3 -> R3C10
- SW60: value R7C4 -> R3C11
- SW61: value R7C5 -> R3C12
- SW62: value R7C6 -> R3C13
- SW63: value R8C0 -> R4C0
- SW64: value R8C1 -> R4C1
- SW65: value R8C2 -> R4C2
- SW66: value R8C3 -> R4C3
- SW67: value R8C4 -> R4C4
- SW68: value R8C5 -> R4C5
- SW69: value R8C6 -> R4C6
- SW70: value R9C0 -> R4C7
- SW71: value R9C1 -> R4C8
- SW72: value R9C2 -> R4C9
- SW73: value R9C3 -> R4C10
- SW74: value R9C4 -> R4C11
- SW75: value R9C5 -> R4C12
- SW76: value R9C6 -> R4C13
- SW77: value R10C0 -> R5C0
- SW78: value R10C1 -> R5C1
- SW79: value R10C2 -> R5C2
- SW80: value R10C3 -> R5C3
- SW81: value R10C4 -> R5C4
- SW82: value R10C5 -> R5C5
- SW83: value R10C6 -> R5C6
- SW84: value R10C7 -> R5C7
- SW85: value R10C8 -> R5C8
- SW86: value R10C9 -> R5C9
- SW9: value R1C0 -> R0C8
